File: PCB/230V.kicad_sch (KiCad schematic)
At the start: 33 parts, among them J12 230V IN, J13 REKU FAN 1, J14 BELIMO, J15 MIX 230V, J16 REKU FAN 2, J17 REKU ZAPAS, K1 Finder 32.21 / 5V, K2 G3MB-202P DC5, K3 G3MB-202P DC5, K4 G3MB-202P DC5, K5 G3MB-202P DC5, Q3 2N3904, Q4 2N3904, Q5 2N3904, Q6 2N3904, Q7 2N3904, U6 IRM-10-5

Commit message: Update PCB to v1.1 and document KiCad project files
Parts:
- C8: footprint Capacitor_SMD:C_0603_1608Metric -> Capacitor_SMD:C_1206_3216Metric
- J12, J13, J16, J17: footprint Connector_Phoenix_GMSTB:PhoenixContact_GMSTBA_2,5_2-G-7,62_1x02_P7.62mm_Horizontal -> Rekuperator:PhoenixContact_MSTBA_2,5_2-G-5,08_1x02_P5.08mm_Horizontal_Edge; MPN 1766233 -> 1757242; MatingConnector GMSTB 2,5/2-ST-7,62 -> MSTB 2,5/2-ST-5,08
- J14, J15: footprint Connector_Phoenix_GMSTB:PhoenixContact_GMSTBA_2,5_3-G-7,62_1x03_P7.62mm_Horizontal -> Rekuperator:PhoenixContact_MSTBA_2,5_3-G-5,08_1x03_P5.08mm_Horizontal_Edge; MPN 1766246 -> 1757255; MatingConnector GMSTB 2,5/3-ST-7,62 -> MSTB 2,5/3-ST-5,08
- R32, R33, R34, R35, R36, R37, R38, R39, R40, R41: footprint Resistor_SMD:R_0603_1608Metric -> Resistor_SMD:R_1206_3216Metric
Other:
- title: (none) -> OpenReku - sterowanie 230 V
