File: PCB/I2C.kicad_sch (KiCad schematic)
At the start: 30 parts, among them J10 CH6 ARK 3.5, J11 CH7 ARK 3.5, J4 CH0 ARK 3.5, J5 CH1 ARK 3.5, J6 CH2 ARK 3.5, J7 CH3 ARK 3.5, J8 CH4 ARK 3.5, J9 CH5 ARK 3.5, U5 TCA9548APWR

Commit message: Update PCB to v1.1 and document KiCad project files
Parts:
- C6, C7: footprint Capacitor_SMD:C_0603_1608Metric -> Capacitor_SMD:C_1206_3216Metric
- J10, J11, J4, J5, J6, J7, J8, J9: footprint Connector_Phoenix_MC:PhoenixContact_MC_1,5_4-G-3.5_1x04_P3.50mm_Horizontal -> Rekuperator:PhoenixContact_MC_1,5_4-G-3.5_1x04_P3.50mm_Horizontal_Edge
- R13, R14, R15, R16, R17, R18, R19, R20, R21, R22, R23, R24, R25, R26, R27, R28, R29, R30, R31: footprint Resistor_SMD:R_0603_1608Metric -> Resistor_SMD:R_1206_3216Metric
Other:
- title: (none) -> OpenReku - multiplekser I2C
