File: PCB/OpenReku.kicad_sch (KiCad schematic)
At the start: 30 parts, among them J1 UART 3V3, J2 FAN1 WYLOT, J3 FAN2 WLOT, Q1 2N3904, Q2 2N3904, SW1 BOOT, SW2 RESET, U1 ESP32-WROOM-32U, U2 LM1117DT-3.3, U3 PC817, U4 PC817

Commit message: Update PCB to v1.1 and document KiCad project files
Parts:
- C3: footprint Capacitor_SMD:C_0603_1608Metric -> Capacitor_SMD:C_1206_3216Metric
- C4, C5: footprint Capacitor_SMD:C_0805_2012Metric -> Capacitor_SMD:C_1206_3216Metric
- R1, R10, R11, R12, R2, R3, R4, R5, R6, R7, R8, R9: footprint Resistor_SMD:R_0603_1608Metric -> Resistor_SMD:R_1206_3216Metric
Other:
- note added: "OpenReku — KONTROLER ESP32"
- note removed: "REKUPERATOR — KONTROLER ESP32"
- title: (none) -> OpenReku - ESP32 / zasilanie / wentylatory
